Commit message: replaced absolute path in env.urdf with relative one

File: wire_sim/config/env.urdf (robot description, URDF)
Before this commit: robot myfirst, 5 links, 4 joints
Links:
- link base_link: geometry visual mesh filename=package://wire_sim/meshes/Stator Stand.STL scale=0.001 0.001 0.001
- link load_cell: geometry visual mesh filename=package://wire_sim/meshes/ATI-9105-NET-DELTA-IP60.STL scale=0.001 0.001 0.001
- link load_cell_plate: geometry visual mesh filename=package://wire_sim/meshes/Load Cell adapter 3d print versio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 scale=0.001 0.001 0.001
